Commit message: Preparing for cartographer test

File: src/bb8/urdf/bb8.urdf.xacro (robot description, xacro)
@@ -38,6 +38,6 @@
         </visual>
     </link>
-    <!-- Laser -->
-    <link name="laser_link"/>
+    <!-- Lidar -->
+    <link name="lidar_link"/>
     <!-- IMU -->
     <link name="imu_link"/>
@@ -51,9 +51,9 @@
         <axis  xyz="0 1 0"/>
         <!-- Limit motion to ±45° -->
-        <limit lower="${-45.0 * pi/180.0}" upper="${45.0 * pi/180.0}"/>
+        <limit lower="${-45.0 * pi/180.0}" upper="${45.0 * pi/180.0}" effort="1.0" velocity="1.0"/>
     </joint>
     <!-- Fixed mount lidar_height above head for lidar, mesh contained in head -->
     <joint name="lidar_joint" type="fixed">
-        <parent link="pitch_link"/>
+        <parent link="head_link"/>
         <child  link="lidar_link"/>
         <origin xyz="0 0 ${lidar_height}" rpy="0 0 0"/>
@@ -61,5 +61,5 @@
     <!-- Fixed mount imu_height above head for imu -->
     <joint name="imu_joint" type="fixed">
-        <parent link="pitch_link"/>
+        <parent link="head_link"/>
         <child  link="imu_link"/>
         <origin xyz="0 0 ${imu_height}" rpy="0 0 0"/>

Commit message: Okay, now we are talking

File: src/bb8/urdf/bb8.urdf.xacro (robot description, xacro)
@@ -39,5 +39,5 @@
     </link>
     <!-- Lidar -->
-    <link name="lidar_link"/>
+    <link name="laser"/>
     <!-- IMU -->
     <link name="imu_link"/>
@@ -56,5 +56,5 @@
     <joint name="lidar_joint" type="fixed">
         <parent link="head_link"/>
-        <child  link="lidar_link"/>
+        <child  link="laser"/>
         <origin xyz="0 0 ${lidar_height}" rpy="0 0 0"/>
     </joint>

Commit message: Now with 100% more IMU

File: src/bb8/urdf/bb8.urdf.xacro (robot description, xacro)
@@ -41,5 +41,5 @@
     <link name="laser"/>
     <!-- IMU -->
-    <link name="imu_link"/>
+    <link name="imu"/>
     <!-- Revolute joint above the sphere: allows pitching only -->
     <joint name="head_joint" type="revolute">
@@ -62,5 +62,5 @@
     <joint name="imu_joint" type="fixed">
         <parent link="head_link"/>
-        <child  link="imu_link"/>
+        <child  link="imu"/>
         <origin xyz="0 0 ${imu_height}" rpy="0 0 0"/>
     </joint>
