Commit message: Update urdf from xarco

File: src/bb8/urdf/bb8.urdf (robot description, URDF)
Before this commit: robot spherical_bot, 4 links, 3 joints
Links:
- removed link imu_link
- added link imu
Joints:
- joint imu_joint: child imu_link -> imu

Commit message: Updated to include sphere_imu

File: src/bb8/urdf/bb8.urdf (robot description, URDF)
Before this commit: robot spherical_bot, 4 links, 3 joints
Links:
- removed link imu
- added link base_footprint; collision cylinder length=0.449 radius=0.165
- added link head_imu
- added link sphere_imu
- link base_link: geometry visual sphere radius=0.165
Joints:
- removed joint imu_joint
- added joint base_joint: type fixed, parent base_footprint, child base_link, origin xyz=0 0 0.165 rpy=0 0 0
- added joint head_imu_joint: type fixed, parent head_link, child head_imu, origin xyz=0 0 0.089 rpy=0 0 0
- added joint sphere_imu_joint: type fixed, parent base_footprint, child sphere_imu, origin xyz=0 0 0.165 rpy=0 0 0
- joint head_joint: origin xyz=0 0 0.165 rpy=0 0 0 -> xyz=0 0 0 rpy=0 0 0
- joint lidar_joint: origin xyz=0 0 0.15 rpy=0 0 0 -> xyz=0 0 0.119 rpy=0 0 0

File: src/bb8/urdf/bb8.urdf.xacro (robot description, xacro)
@@ -1,9 +1,22 @@
 <?xml version="1.0"?>
-<robot xmlns:xacro="http://www.ros.org/wiki/xacro" name="spherical_bot">
+<robot xmlns:xacro="http://www.ros.org/wiki/xacro" name="ORBIT">
     <xacro:property name="sphere_diameter" value="0.33"/>
-    <xacro:property name="lidar_height" value="0.15"/>
-    <xacro:property name="imu_height" value="0.13"/>
-    <xacro:property name="mass" value="2"/>
-    <!-- Base Sphere -->
+    <xacro:property name="head_diameter" value="${sphere_diameter / 2}"/>
+    <xacro:property name="mass" value="10"/>
+    <!-- From base_footprint -->
+    <xacro:property name="head_revolution_height" value="${sphere_diameter / 2}"/>
+    <xacro:property name="sphere_imu_height" value="${sphere_diameter / 2}"/>
+    <!-- From head_link -->
+    <xacro:property name="head_imu_height" value="0.089"/>
+    <xacro:property name="lidar_height" value="0.119"/>
+    <!-- Fottprint, bottom of the sphere, contact point with the terrain -->
+    <link name="base_footprint">
+        <collision>
+            <geometry>
+                <cylinder length="${sphere_diameter + lidar_height}" radius="${sphere_diameter / 2}"/>
+            </geometry>
+        </collision>
+    </link>
+    <!-- Center of the sphere, revolution center point for the head -->
     <link name="base_link">
         <visual>
@@ -18,11 +31,6 @@
             </geometry> -->
         </visual>
-        <collision>
-            <geometry>
-                <cylinder length="${sphere_diameter + lidar_height}" radius="${sphere_diameter / 2}"/>
-            </geometry>
-        </collision>
     </link>
-    <!-- Head, mesh contains lidar -->
+    <!-- Head base, point where the middle of the head "touches" the sphere -->
     <link name="head_link">
         <visual>
@@ -38,8 +46,22 @@
         </visual>
     </link>
+    <!-- IMU in the sphere -->
+    <link name="sphere_imu"/>
     <!-- Lidar -->
     <link name="laser"/>
-    <!-- IMU -->
-    <link name="imu"/>
+    <!-- IMU in the head -->
+    <link name="head_imu"/>
+    <!-- Revolution center point for the head -->
+    <joint name="base_joint" type="fixed">
+        <parent link="base_footprint"/>
+        <child  link="base_link"/>
+        <origin xyz="0 0 ${head_revolution_height}" rpy="0 0 0"/>
+    </joint>
+    <!-- Fixed mount sphere IMU -->
+    <joint name="sphere_imu_joint" type="fixed">
+        <parent link="base_footprint"/>
+        <child  link="sphere_imu"/>
+        <origin xyz="0 0 ${sphere_imu_height}" rpy="0 0 0"/>
+    </joint>
     <!-- Revolute joint above the sphere: allows pitching only -->
     <joint name="head_joint" type="revolute">
@@ -47,11 +69,11 @@
         <child  link="head_link"/>
         <!-- Offset joint pivot radius above base center -->
-        <origin xyz="0 0 ${sphere_diameter / 2}" rpy="0 0 0"/>
+        <origin xyz="0 0 0" rpy="0 0 0"/>
         <!-- Axis along Y for forward/back tilt -->
         <axis  xyz="0 1 0"/>
         <!-- Limit motion to ±45° -->
-        <limit lower="${-45.0 * pi/180.0}" upper="${45.0 * pi/180.0}" effort="1.0" velocity="1.0"/>
+        <limit lower="${-45.0 * pi / 180.0}" upper="${45.0 * pi / 180.0}" effort="1.0" velocity="1.0"/>
     </joint>
-    <!-- Fixed mount lidar_height above head for lidar, mesh contained in head -->
+    <!-- Fixed mount lidar_height above head for lidar -->
     <joint name="lidar_joint" type="fixed">
         <parent link="head_link"/>
@@ -59,9 +81,9 @@
         <origin xyz="0 0 ${lidar_height}" rpy="0 0 0"/>
     </joint>
-    <!-- Fixed mount imu_height above head for imu -->
-    <joint name="imu_joint" type="fixed">
+    <!-- Fixed mount head_imu_height above head for imu -->
+    <joint name="head_imu_joint" type="fixed">
         <parent link="head_link"/>
-        <child  link="imu"/>
-        <origin xyz="0 0 ${imu_height}" rpy="0 0 0"/>
+        <child  link="head_imu"/>
+        <origin xyz="0 0 ${head_imu_height}" rpy="0 0 0"/>
     </joint>
 </robot>

Commit message: New Servo joint

File: src/bb8/urdf/bb8.urdf (robot description, URDF)
Before this commit: robot ORBIT, 6 links, 5 joints
Links:
- added link servo_link
Joints:
- joint head_joint: axis 0 1 0 -> (none); limit lower=-0.7853981633974483 upper=0.7853981633974483 effort=1.0 velocity=1.0 -> (none); origin xyz=0 0 0 rpy=0 0 0 -> xyz=0 0 0.165 rpy=0 0 0; parent base_link -> servo_link; type revolute -> fixed

File: src/bb8/urdf/bb8.urdf.xacro (robot description, xacro)
@@ -18,5 +18,5 @@
         </collision>
     </link>
-    <!-- Center of the sphere, revolution center point for the head -->
+    <!-- Center of the sphere, revolution pivit point for the head -->
     <link name="base_link">
         <visual>
@@ -32,4 +32,6 @@
         </visual>
     </link>
+    <!-- Servo link, revolution for the head -->
+    <link name="servo_link"/>
     <!-- Head base, point where the middle of the head "touches" the sphere -->
     <link name="head_link">
@@ -64,8 +66,8 @@
         <origin xyz="0 0 ${sphere_imu_height}" rpy="0 0 0"/>
     </joint>
-    <!-- Revolute joint above the sphere: allows pitching only -->
+    <!-- Revolute joint of the sphere: allows pitching only -->
     <joint name="head_joint" type="revolute">
         <parent link="base_link"/>
-        <child  link="head_link"/>
+        <child  link="servo_link"/>
         <!-- Offset joint pivot radius above base center -->
         <origin xyz="0 0 0" rpy="0 0 0"/>
@@ -74,4 +76,10 @@
         <!-- Limit motion to ±45° -->
         <limit lower="${-45.0 * pi / 180.0}" upper="${45.0 * pi / 180.0}" effort="1.0" velocity="1.0"/>
+    </joint>
+    <!-- Head link: Lenght of the servo link -->
+    <joint name="head_joint" type="fixed">
+        <parent link="servo_link"/>
+        <child  link="head_link"/>
+        <origin xyz="0 0 ${sphere_diameter / 2}" rpy="0 0 0"/>
     </joint>
     <!-- Fixed mount lidar_height above head for lidar -->

Commit message: MANAUL working - Remote

File: src/bb8/urdf/bb8.urdf (robot description, URDF)
Before this commit: robot ORBIT, 7 links, 5 joints
Joints:
- added joint servo_joint: type revolute, parent base_link, child servo_link, origin xyz=0 0 0 rpy=0 0 0, axis 0 1 0, limit lower=-0.7853981633974483 upper=0.7853981633974483 effort=1.0 velocity=1.0

File: src/bb8/urdf/bb8.urdf.xacro (robot description, xacro)
@@ -67,5 +67,5 @@
     </joint>
     <!-- Revolute joint of the sphere: allows pitching only -->
-    <joint name="head_joint" type="revolute">
+    <joint name="servo_joint" type="revolute">
         <parent link="base_link"/>
         <child  link="servo_link"/>
